File: pcb/basic_R/keyboard-layouter-playground.kicad_pcb (KiCad board)
At the start: 2 copper layers, 243 x 151.8 mm, 129 parts, among them J2 MJ-4PP-9, SW103 SW_Push, SW104 SW_Push, SW105 SW_Push, SW202 SW_Push, SW303 SW_Push, SW305 SW_Push, SW31 SW_Push, SW32 SW_Push, SW33 SW_Push, SW34 SW_Push, SW35 SW_Push, SW36 SW_Push, SW37 SW_Push, SW38 SW_Push, SW39 SW_Push, SW40 SW_Push, SW41 SW_Push, SW42 SW_Push, SW43 SW_Push, SW44 SW_Push, SW45 SW_Push, SW46 SW_Push, SW47 SW_Push, SW48 SW_Push, SW49 SW_Push, SW50 SW_Push, SW51 SW_Push, SW52 SW_Push, SW53 SW_Push, SW54 SW_Push, SW55 SW_Push, SW56 SW_Push, SW57 SW_Push, SW58 SW_Push, SW59 SW_Push, SW60 SW_Push, SW61 SW_Push, SW62 SW_Push, SW63 SW_Push, SW64 SW_Push, SW65 SW_Push, SW66 SW_Push, SW67 SW_Push, SW68 SW_Push, SW69 SW_Push, SW70 SW_Push, SW71 SW_Push, SW72 SW_Push, SW73 SW_Push, SW74 SW_Push, SW75 SW_Push, SW76 SW_Push, SW77 SW_Push, SW78 SW_Push, SW79 SW_Push, SW80 SW_Push, SW81 SW_Push, SW82 SW_Push, SW83 SW_Push, SW84 SW_Push, SW85 SW_Push, SW901 SW_Push, U2 Elite-C

Commit message: left promicro both OK.
Parts:
- moved R2 4.45 mm to (241.0, 107.5), turned to 0 degrees
- turned R1 to 0 degrees
Routing:
- net SDA2: track 234.1 -> 242.1 mm
- net Net-(J2-PadD): track 232.8 -> 238.3 mm
- net Net-(J2-PadB): track 273.8 -> 270.1 mm

Commit message: bugfix
Parts:
- added TPH: MountingHole_3.5mm, MountingHole:MountingHole_3.5mm, F.Cu at (24.4, 194.7)
- SW901: footprint gammy:SW_Cherry_MX_ISOEnter_Plate -> gammy:SW_Cherry_MX_ISOEnter_Stabilizer_5pin
- moved D901 13.8 mm to (176.3, 198.4), turned to 0 degrees
Routing:
- net COL16: track 199.9 -> 221.9 mm
- net Net-(D901-Pad1): track 24.1 -> 35.6 mm
- net row10: track 330.2 -> 332.9 mm
- net COL9: track 342.1 -> 343.8 mm
- net COL11: track 309.8 -> 309.1 mm
- net COL12: track 254.8 -> 254.1 mm
- net COL14: track 235.8 -> 235.1 mm
- net COL15: track 214.9 -> 214.2 mm
- net COL17: track 82.9 -> 82.2 mm
