File: pcb/basic_L/keyboard-layouter-playground.kicad_pcb (KiCad board)
At the start: 2 copper layers, 138 x 151.8 mm, 71 parts, among them J1 MJ-4PP-9, SW10 SW_Push, SW101 SW_Push, SW102 SW_Push, SW11 SW_Push, SW12 SW_Push, SW13 SW_Push, SW14 SW_Push, SW15 SW_Push, SW16 SW_Push, SW17 SW_Push, SW18 SW_Push, SW19 SW_Push, SW20 SW_Push, SW201 SW_Push, SW21 SW_Push, SW22 SW_Push, SW23 SW_Push, SW24 SW_Push, SW25 SW_Push, SW26 SW_Push, SW27 SW_Push, SW28 SW_Push, SW29 SW_Push, SW3 SW_Push, SW30 SW_Push, SW301 SW_Push, SW302 SW_Push, SW304 SW_Push, SW4 SW_Push, SW5 SW_Push, SW6 SW_Push, SW601 SW_Push, SW7 SW_Push, U1 Elite-C-keebio

Commit message: left promicro both OK.
Parts:
- moved R1 0.50 mm to (144.2, 121.3)
- moved R2 0.50 mm to (144.2, 116.5)
Connections:
- U1 pad 13: COL5 -> row1
- U1 pad 14: (no net) -> COL1
- U1 pad 15: (no net) -> COL2
- U1 pad 18: (no net) -> COL3
- U1 pad 19: (no net) -> COL4
- U1 pad 20: (no net) -> COL5
- U1 pad 25: row1 -> (no net)
- U1 pad 26: COL1 -> (no net)
- U1 pad 27: COL2 -> (no net)
- U1 pad 28: COL3 -> (no net)
- U1 pad 29: COL4 -> (no net)
Routing:
- net COL4: track 210.6 -> 230.9 mm
- net COL3: track 184.2 -> 203.0 mm
- net COL5: track 221.7 -> 240.5 mm
- net COL1: track 122.9 -> 139.1 mm, vias 0 -> 2
- net COL2: track 133.1 -> 146.4 mm, vias 0 -> 1
- net row1: track 148.6 -> 157.1 mm
- net VCC: track 144.0 -> 147.5 mm
- net Net-(J1-PadD): track 142.7 -> 141.3 mm
- net SDA1: track 145.9 -> 145.2 mm

Commit message: bugfix
Connections:
- U1 pad 17: (no net) -> COL3
- U1 pad 18: COL3 -> COL4
- U1 pad 19: COL4 -> COL5
- U1 pad 20: COL5 -> (no net)
Routing:
- net COL3: track 203.0 -> 219.2 mm, vias 0 -> 1
- net COL4: track 230.9 -> 216.6 mm
- net COL5: track 240.5 -> 228.2 mm
- net COL1: track 139.1 -> 132.0 mm, vias 2 -> 1
- net COL2: track 146.4 -> 140.4 mm, vias 1 -> 0
- net Net-(J1-PadD): track 141.3 -> 145.3 mm
- net COL0: track 138.7 -> 135.2 mm
- net row1: track 157.1 -> 160.0 mm
- net GND: track 147.7 -> 149.7 mm
